Commit message: Minor formatting changes to urdf description

File: urdf/roboclaw_description.urdf.xacro (robot description, xacro)
@@ -100,6 +100,6 @@
           iyy="${wheel_mass / 12.0 * wheel_radius*wheel_radius}" iyz="0.0"
           izz="${wheel_mass / 12.0 * wheel_radius*wheel_radius}"/>
-        </inertial>
-      </link>
+      </inertial>
+    </link>
     <joint name="caster_left_wheel_joint" type="fixed">
       <parent link="base_link"/>
